File: Controller_PCB/230V_controller.kicad_pcb (KiCad board)
At the start: 2 copper layers, 0 parts

Commit message: Added PCB Design
Parts:
- added A1: Arduino_Nano_v3.x, Module:Arduino_Nano, F.Cu at (194.6, 93.5)
- added D1: 1N4007, Diode_THT:D_DO-41_SOD81_P10.16mm_Horizontal, F.Cu at (226.9, 74.0)
- added D2: 1N4007, Diode_THT:D_DO-41_SOD81_P10.16mm_Horizontal, F.Cu at (252.1, 74.0)
- added D3: 1N4007, Diode_THT:D_DO-41_SOD81_P10.16mm_Horizontal, F.Cu at (237.1, 78.5)
- added D4: 1N4007, Diode_THT:D_DO-41_SOD81_P10.16mm_Horizontal, F.Cu at (241.9, 78.5)
- added D5: LED, LED_THT:LED_D3.0mm, F.Cu at (216.0, 118.5)
- added D6: LED, LED_THT:LED_D3.0mm, F.Cu at (216.0, 106.5)
- added D7: 1N4148, Diode_THT:D_DO-35_SOD27_P7.62mm_Horizontal, F.Cu at (216.8, 111.0)
- added D8: 1N4148, Diode_THT:D_DO-35_SOD27_P7.62mm_Horizontal, F.Cu at (219.7, 93.0)
- added D9: LED, LED_THT:LED_D3.0mm, F.Cu at (181.4, 135.0)
- added J1: Screw_Terminal_01x02, TerminalBlock_Phoenix:TerminalBlock_Phoenix_MKDS-1,5-2_1x02_P5.00mm_Horizontal, F.Cu at (242.0, 54.0)
- added J2: Screw_Terminal_01x02, TerminalBlock_Phoenix:TerminalBlock_Phoenix_MKDS-1,5-2_1x02_P5.00mm_Horizontal, F.Cu at (246.5, 130.0)
- added J3: Screw_Terminal_01x02, TerminalBlock_Phoenix:TerminalBlock_Phoenix_MKDS-1,5-2_1x02_P5.00mm_Horizontal, F.Cu at (246.5, 117.0)
- added J4: Screw_Terminal_01x02, TerminalBlock_Phoenix:TerminalBlock_Phoenix_MKDS-1,5-2_1x02_P5.00mm_Horizontal, F.Cu at (246.3, 104.0)
- added K1: HF32FA, My_Footprints:HF32FA_Type1_FormC, F.Cu at (219.2, 119.8)
- added K2: HF32FA, My_Footprints:HF32FA_Type1_FormC, F.Cu at (219.2, 107.0)
- added Q1: BC546, Package_TO_SOT_THT:TO-92_Inline_Wide, F.Cu at (210.0, 114.0)
- added Q2: BC546, Package_TO_SOT_THT:TO-92_Inline_Wide, F.Cu at (211.0, 98.5)
- added Q3: BT136-600, Package_TO_SOT_THT:TO-220-3_Vertical, F.Cu at (235.0, 141.0)
- added Q4: BC546, Package_TO_SOT_THT:TO-92_Inline_Wide, F.Cu at (186.5, 135.4)
- added R1: 47k, Resistor_THT:R_Axial_DIN0207_L6.3mm_D2.5mm_P10.16mm_Horizontal, F.Cu at (236.6, 66.5)
- added R10: 2.2k, Resistor_THT:R_Axial_DIN0207_L6.3mm_D2.5mm_P10.16mm_Horizontal, F.Cu at (189.1, 118.9)
- added R11: 330, Resistor_THT:R_Axial_DIN0207_L6.3mm_D2.5mm_P10.16mm_Horizontal, F.Cu at (179.5, 118.9)
- added R2: 47k, Resistor_THT:R_Axial_DIN0207_L6.3mm_D2.5mm_P10.16mm_Horizontal, F.Cu at (241.8, 66.5)
- added R3: 10k, Resistor_THT:R_Axial_DIN0207_L6.3mm_D2.5mm_P10.16mm_Horizontal, F.Cu at (219.6, 89.5)
- added R4: 330, Resistor_THT:R_Axial_DIN0207_L6.3mm_D2.5mm_P10.16mm_Horizontal, F.Cu at (198.0, 113.9)
- added R5: 220, Resistor_THT:R_Axial_DIN0207_L6.3mm_D2.5mm_P10.16mm_Horizontal, F.Cu at (196.4, 140.5)
- added R6: 330, Resistor_THT:R_Axial_DIN0207_L6.3mm_D2.5mm_P10.16mm_Horizontal, F.Cu at (203.5, 124.6)
- added R7: 2.2k, Resistor_THT:R_Axial_DIN0207_L6.3mm_D2.5mm_P10.16mm_Horizontal, F.Cu at (198.0, 97.9)
- added R8: 2.2k, Resistor_THT:R_Axial_DIN0207_L6.3mm_D2.5mm_P10.16mm_Horizontal, F.Cu at (203.5, 97.9)
- added R9: 220, Resistor_THT:R_Axial_DIN0207_L6.3mm_D2.5mm_P10.16mm_Horizontal, F.Cu at (217.9, 128.0)
- added REF**: MountingHole_2.5mm, MountingHole:MountingHole_2.5mm, F.Cu at (254.0, 144.0)
- added REF**: MountingHole_2.5mm, MountingHole:MountingHole_2.5mm, F.Cu at (178.0, 144.0)
- added REF**: MountingHole_2.5mm, MountingHole:MountingHole_2.5mm, F.Cu at (254.0, 46.0)
- added REF**: MountingHole_2.5mm, MountingHole:MountingHole_2.5mm, F.Cu at (178.0, 46.0)
- added SW2: SW_Push_DPDT, Button_Switch_THT:SW_Push_2P2T_Toggle_CK_PVA2xxH1xxxxxxV2, F.Cu at (181.0, 101.0)
- added U1: PC817, Package_DIP:DIP-4_W7.62mm, F.Cu at (234.3, 86.3)
- added U3: MOC3021M, Package_DIP:DIP-6_W7.62mm, F.Cu at (222.3, 140.5)
Routing:
- net GND: track 0.00 -> 351.8 mm
- net DIMM_TRIAC: track 0.00 -> 140.8 mm
- net RELAY_2: track 0.00 -> 112.5 mm
- net unconnected-(A1-D3-Pad6): track 0.00 -> 112.0 mm
- net L1: track 0.00 -> 104.6 mm
- net +5V: track 0.00 -> 97.2 mm
- net NEUTRAL: track 0.00 -> 81.3 mm
- net DIMMER_EN: track 0.00 -> 66.7 mm
- net RELAY_1: track 0.00 -> 63.7 mm
- net Net-(Q4-C): track 0.00 -> 55.2 mm
- net ZCD: track 0.00 -> 37.2 mm
- net Net-(D8-A): track 0.00 -> 29.5 mm
- net Net-(Q3-G): track 0.00 -> 24.9 mm
- net Net-(R5-Pad2): track 0.00 -> 23.9 mm
- net Net-(D5-A): track 0.00 -> 21.9 mm
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- added copper zone on B.Cu, net GND
- added copper zone on F.Cu, net GND
Other:
- board outline added: 85 x 106.5 mm
- board text added: "(L) DIMMER (N)"
- board text added: "(L) RELAY 1 (N)"
- board text added: "(L) RELAY 2 (N)"
- board text added: "(N) MAINS INPUT (L)"
- board text added: "----------------- Mains Voltage Device Controller ----------------- by: Konrad Korzeniowski 08.08.2024"
- board text added: "CONNECT TO PC"
- board text added: "DIMMER ENABLED"
- board text added: "K1"
