File: Controller_PCB/230V_controller.kicad_sch (KiCad schematic)
At the start: 34 parts, among them J1 Screw_Terminal_01x02, J2 Screw_Terminal_01x02, J3 Screw_Terminal_01x02, J4 Screw_Terminal_01x02, K1 HF32FA, K2 HF32FA, Q1 BC546, Q2 BC546, Q3 BT136-600, Q4 BC546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

Commit message: A little schematic update Nothing to worry about :) (I just don't remeber what I've changed)
Other:
- note added: "Bistable Relay 1"
- note added: "Bistable Relay 2"
- note removed: "Bistable Relay 1 Single Isolation"
- note removed: "Bistable Relay 2 Double Isolation"
Changed lines of the file:
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@@
 		)
 	)
-	(text "Bistable Relay 1\nSingle Isolation"
+	(text "Bistable Relay 1\n"
 		(exclude_from_sim no)
-		(at 163.83 62.23 0)
+		(at 163.322 60.198 0)
 		(effects
 			(font
@@
 		)
 	)
-	(text "Bistable Relay 2\nDouble Isolation"
+	(text "Bistable Relay 2"
 		(exclude_from_sim no)
-		(at 163.83 106.68 0)
+		(at 163.322 104.394 0)
 		(effects
 			(font

Commit message: Added PCB Design
Connections:
- net GND: now also SW2.1 (A), SW2.2 (B), SW2.3 (C), SW2.4 (A)
- no-connect marks 28 -> 23
Changed lines of the file:
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@@
+	)
+	(junction
+		(at 50.8 85.09)
+		(diameter 0)
+		(color 0 0 0 0)
 	)
 	(junction
@@
 	)
 	(junction
+		(at 60.96 77.47)
+		(diameter 0)
+		(color 0 0 0 0)
+	)
+	(junction
+		(at 60.96 72.39)
+		(diameter 0)
+		(color 0 0 0 0)
+	)
+	(junction
 		(at 104.14 44.45)
 		(diameter 0)
@@
 	)
 	(no_connect
-		(at 50.8 74.93)
-	)
-	(no_connect
 		(at 77.47 82.55)
 	)
@@
 	)
 	(no_connect
-		(at 77.47 87.63)
-	)
-	(no_connect
 		(at 102.87 97.79)
 	)
@@
 	)
 	(no_connect
-		(at 60.96 82.55)
-	)
-	(no_connect
-		(at 60.96 77.47)
-	)
-	(no_connect
 		(at 240.03 110.49)
 	)
@@
 	)
 	(no_connect
-		(at 60.96 72.39)
-	)
-	(no_connect
 		(at 77.47 110.49)
 	)
@@
 	(wire
 		(pts
+			(xy 60.96 72.39) (xy 60.96 77.47)
+		)
+		(stroke
+			(width 0)
+			(type default)
+		)
+	)
+	(wire
+		(pts
 			(xy 45.72 22.86) (xy 45.72 25.4)
 		)
@@
 	(wire
 		(pts
+			(xy 60.96 77.47) (xy 60.96 82.55)
+		)
+		(stroke
+			(width 0)
+			(type default)
+		)
+	)
+	(wire
+		(pts
 			(xy 48.26 86.36) (xy 48.26 85.09)
 		)
@@
 	(wire
 		(pts
+			(xy 60.96 72.39) (xy 66.04 72.39)
+		)
+		(stroke
+			(width 0)
+			(type default)
+		)
+	)
+	(wire
+		(pts
 			(xy 137.16 43.18) (xy 137.16 45.72)
 		)
@@
 	(wire
 		(pts
+			(xy 66.04 72.39) (xy 66.04 73.66)
+		)
+		(stroke
+			(width 0)
+			(type default)
+		)
+	)
+	(wire
+		(pts
 			(xy 224.79 86.36) (xy 226.06 86.36)
 		)
@@
 			(width 0)
 			(type dash_dot_dot)
+		)
+	)
+	(wire
+		(pts
+			(xy 50.8 74.93) (xy 50.8 85.09)
+		)
+		(stroke
+			(width 0)
+			(type default)
 		)
 	)
@@
 					(unit 1)
 				)
+			)
+		)
+	)
+	(symbol
+		(lib_id "power:GND")
+		(at 66.04 73.66 0)
+		(unit 1)
+		(exclude_from_sim no)
+		(in_bom yes)
+		(on_board yes)
+		(dnp no)
+		(fields_autoplaced yes)
+		(property "Reference" "#PWR09"
+			(at 66.04 80.01 0)
+			(effects
+				(font
+					(size 1.27 1.27)
+				)
+				(hide yes)
+			)
+		)
+		(property "Value" "GND"
+			(at 66.04 78.74 0)
+			(effects
+				(font
+					(size 1.27 1.27)
+				)
+			)
+		)
+		(property "Footprint" ""
+			(at 66.04 73.66 0)
+			(effects
+				(font
+					(size 1.27 1.27)
+				)
+				(hide yes)
+			)
+		)
+		(property "Datasheet" ""
+			(at 66.04 73.66 0)
+			(effects
+				(font
+					(size 1.27 1.27)
+				)
+				(hide yes)
+			)
+		)
+		(property "Description" ""
+			(at 66.04 73.66 0)
+			(effects
+				(font
+					(size 1.27 1.27)
+				)
+				(hide yes)
+			)
+		)
+		(pin "1"
+		)
+		(instances
+			(project "230V_controller"
+				(path "/0518519f-5f34-4fd9-905a-d6a5ef6e19ea"
+					(reference "#PWR09")
+					(unit 1)
+				)
